File: eeprom_shield.kicad_pcb (KiCad board)
At the start: 2 copper layers, 43.2 x 58.4 mm, 9 parts, among them J1 Conn_02x20_Odd_Even, J2 Conn_02x16_Odd_Even, U1 SST39SF040

Commit message: Comments added
Other:
- board text added: "Power"
- board text added: "Read"
- board text added: "Write"
Changed lines of the file:
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@@
     (effects (font (size 2 2) (thickness 0.15)) (justify mirror))
   )
+  (gr_text "Power" (at 100.426487 64.135) (layer "F.SilkS")
+    (effects (font (size 1 1) (thickness 0.15)))
+  )
   (gr_text "V1.0" (at 68.58 52.720103) (layer "F.SilkS")
+    (effects (font (size 1 1) (thickness 0.15)))
+  )
+  (gr_text "Write" (at 92.71 64.135) (layer "F.SilkS")
     (effects (font (size 1 1) (thickness 0.15)))
   )
@@
     (effects (font (size 1 1) (thickness 0.15) italic))
   )
+  (gr_text "Read" (at 92.71 57.15) (layer "F.SilkS")
+    (effects (font (size 1 1) (thickness 0.15)))
+  )
   (segment (start 92.71 67.31) (end 93.985 67.31) (width 0.25) (layer "B.Cu") (net 1))
