File: eeprom_shield.kicad_sch (KiCad schematic)
At the start: 9 parts, among them J1 Conn_02x20_Odd_Even, J2 Conn_02x16_Odd_Even, U1 SST39SF040

Commit message: Comments added
Connections:
- net at U1.24 (OE): now also J1.29 (Pin_29)
Other:
- company: (none) -> VarioStudio
- title: (none) -> EEPROM shield
Changed lines of the file:
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@@
 (kicad_sch (version 20211123) (generator eeschema)
   (paper "A4")
+  (title_block
+    (title "EEPROM shield")
+    (rev "1.0")
+    (company "VarioStudio")
+    (comment 1 "D1 - power LED")
+    (comment 2 "D2 - read LED")
+    (comment 3 "D3 - write LED")
+    (comment 4 "R1,R2,R3 - 220...1K")
+  )
   (junction (at 69.85 22.86) (diameter 0) (color 0 0 0 0)
   )
@@
     (stroke (width 0) (type default) (color 0 0 0 0))
   )
+  (wire (pts (xy 74.93 87.63) (xy 82.55 87.63))
+    (stroke (width 0) (type default) (color 0 0 0 0))
+  )
   (wire (pts (xy 67.31 31.75) (xy 115.57 31.75))
     (stroke (width 0) (type default) (color 0 0 0 0))
@@
     (stroke (width 0) (type default) (color 0 0 0 0))
   )
+  (wire (pts (xy 74.93 116.84) (xy 74.93 87.63))
+    (stroke (width 0) (type default) (color 0 0 0 0))
+  )
   (wire (pts (xy 82.55 64.77) (xy 77.47 64.77))
     (stroke (width 0) (type default) (color 0 0 0 0))
@@
     (stroke (width 0) (type default) (color 0 0 0 0))
   )
+  (wire (pts (xy 125.73 116.84) (xy 74.93 116.84))
+    (stroke (width 0) (type default) (color 0 0 0 0))
+  )
